File: flicker_stitch.kicad_sch (KiCad schematic)
At the start: 0 parts

Commit message: demo resistor
Parts:
- added H1, H2: MountingHole_Pad, MountingHole:MountingHole_2.2mm_M2_DIN965_Pad, symbol Mechanical:MountingHole_Pad
- added R1: N/A, Resistor_SMD:R_0805_2012Metric, symbol Device:R_US
Connections:
- new net: H1.1, R1.1
- new net: H2.1, R1.2
