File: fs_resistor_0805/fs_resistor_0805.kicad_sch (KiCad schematic)
At the start: 3 parts

Commit message: first draft of 0805 breakout board
Other:
- company: (none) -> Flicker Stitch
- title: (none) -> resistor 0805 stitch breakout board
Changed lines of the file:
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@@
 	(generator_version "10.0")
 	(paper "A4")
+	(title_block
+		(title "resistor 0805 stitch breakout board")
+		(date "2026-03-24")
+		(rev "r1")
+		(company "Flicker Stitch")
+	)
 	(wire
 		(pts
@@
 		)
 		(instances
-			(project "flicker_stitch"
+			(project "fs_resistor_0805"
 				(path "/2e247ec3-ce3e-43b1-b05f-8a11fd5b17f6"
 					(reference "R1")
@@
 		)
 		(instances
-			(project "flicker_stitch"
+			(project "fs_resistor_0805"
 				(path "/2e247ec3-ce3e-43b1-b05f-8a11fd5b17f6"
 					(reference "H2")
@@
 		)
 		(instances
-			(project "flicker_stitch"
+			(project "fs_resistor_0805"
 				(path "/2e247ec3-ce3e-43b1-b05f-8a11fd5b17f6"
 					(reference "H1")

Commit message: add hand soldering pad
Parts:
- H2: footprint MountingHole:MountingHole_2.2mm_M2_DIN965_Pad -> MountingHole:MountingHole_2.2mm_M2_DIN965_Pad_TopBottom
- R1: footprint Resistor_SMD:R_0805_2012Metric -> Resistor_SMD:R_0805_2012Metric_Pad1.20x1.40mm_HandSolder
Changed lines of the file:
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@@
 			)
 		)
-		(property "Footprint" "Resistor_SMD:R_0805_2012Metric"
+		(property "Footprint" "Resistor_SMD:R_0805_2012Metric_Pad1.20x1.40mm_HandSolder"
 			(at 114.046 68.834 90)
 			(hide yes)
@@
 			)
 		)
-		(property "Footprint" "MountingHole:MountingHole_2.2mm_M2_DIN965_Pad"
+		(property "Footprint" "MountingHole:MountingHole_2.2mm_M2_DIN965_Pad_TopBottom"
 			(at 113.03 82.55 0)
 			(hide yes)
